File: granite.sch (KiCad schematic (older format))
At the start: 29 parts, among them CON1 USB-MINI-B WM17115-ND, IC1 ATMEGA32U4, SW1 SW_PUSH, Y1 16MHz

Commit message: update schematic and add pcb
Parts:
- removed Y1: 16MHz, Crystals:Crystal_HC49-SD_SMD, symbol Crystal
- added Y1: ABM8G, bwu-keyboard:bwu-ABM8G-16.000MHZ-4Y-T3, symbol ABM8G
- C6, C8: value 1uF -> 1µF
- R1, R2: value 22 -> 22Ω
- R3: value 1K -> 1kΩ
- S0:0, S0:1, S0:2, S1:0, S1:1, S1:2: footprint CHERRY_PCB_100H:CHERRY_PCB_100H -> bwu-keyboard:bwu-mx1a-1u
- S2:1: footprint CHERRY_PCB_100H:CHERRY_PCB_100H -> bwu-keyboard:bwu-mx1a-2u
Connections:
- wire segments 103 -> 107
Other:
- moved on the sheet: C4, C5
Changed lines of the file:
@@
 P 2750 6850
 F 0 "C6" H 2775 6950 50  0000 L CNN
-F 1 "1uF" H 2775 6750 50  0000 L CNN
+F 1 "1µF" H 2775 6750 50  0000 L CNN
 F 2 "Capacitors_SMD:C_0805_HandSoldering" H 2750 6850 60  0001 C CNN
 F 3 "" H 2750 6850 60  0000 C CNN
@@
 P 2950 6300
 F 0 "R2" V 3030 6300 50  0000 C CNN
-F 1 "22" V 2950 6300 50  0000 C CNN
+F 1 "22Ω" V 2950 6300 50  0000 C CNN
 F 2 "Resistors_SMD:R_0805_HandSoldering" V 2880 6300 30  0001 C CNN
 F 3 "" H 2950 6300 30  0000 C CNN
@@
 P 2950 6100
 F 0 "R1" V 3030 6100 50  0000 C CNN
-F 1 "22" V 2950 6100 50  0000 C CNN
+F 1 "22Ω" V 2950 6100 50  0000 C CNN
 F 2 "Resistors_SMD:R_0805_HandSoldering" V 2880 6100 30  0001 C CNN
 F 3 "" H 2950 6100 30  0000 C CNN
@@
 $EndComp
 $Comp
-L Crystal Y1
-U 1 1 559D400C
-P 2400 4600
-F 0 "Y1" H 2400 4750 50  0000 C CNN
-F 1 "16MHz" H 2400 4450 50  0000 C CNN
-F 2 "Crystals:Crystal_HC49-SD_SMD" H 2400 4600 60  0001 C CNN
-F 3 "" H 2400 4600 60  0000 C CNN
-	1    2400 4600
-	1    0    0    -1
-$EndComp
-$Comp
 L CP1 C4
 U 1 1 559D7687
-P 2100 4900
-F 0 "C4" H 2125 5000 50  0000 L CNN
-F 1 "10pF" H 2125 4800 50  0000 L CNN
-F 2 "Capacitors_SMD:C_0805_HandSoldering" H 2100 4900 60  0001 C CNN
-F 3 "" H 2100 4900 60  0000 C CNN
-	1    2100 4900
+P 1650 4950
+F 0 "C4" H 1675 5050 50  0000 L CNN
+F 1 "10pF" H 1675 4850 50  0000 L CNN
+F 2 "Capacitors_SMD:C_0805_HandSoldering" H 1650 4950 60  0001 C CNN
+F 3 "" H 1650 4950 60  0000 C CNN
+	1    1650 4950
 	1    0    0    -1
 $EndComp
@@
 L CP1 C5
 U 1 1 559D7752
-P 2700 4900
-F 0 "C5" H 2725 5000 50  0000 L CNN
-F 1 "10pF" H 2725 4800 50  0000 L CNN
-F 2 "Capacitors_SMD:C_0805_HandSoldering" H 2700 4900 60  0001 C CNN
-F 3 "" H 2700 4900 60  0000 C CNN
-	1    2700 4900
+P 3000 4950
+F 0 "C5" H 3025 5050 50  0000 L CNN
+F 1 "10pF" H 3025 4850 50  0000 L CNN
+F 2 "Capacitors_SMD:C_0805_HandSoldering" H 3000 4950 60  0001 C CNN
+F 3 "" H 3000 4950 60  0000 C CNN
+	1    3000 4950
 	1    0    0    -1
 $EndComp
@@
 L GNDREF #PWR06
 U 1 1 559D780C
-P 2700 5200
-F 0 "#PWR06" H 2700 4950 60  0001 C CNN
-F 1 "GNDREF" H 2700 5050 60  0000 C CNN
-F 2 "" H 2700 5200 60  0000 C CNN
-F 3 "" H 2700 5200 60  0000 C CNN
-	1    2700 5200
+P 3000 5200
+F 0 "#PWR06" H 3000 4950 60  0001 C CNN
+F 1 "GNDREF" H 3000 5050 60  0000 C CNN
+F 2 "" H 3000 5200 60  0000 C CNN
+F 3 "" H 3000 5200 60  0000 C CNN
+	1    3000 5200
 	1    0    0    -1
 $EndComp
@@
 L GNDREF #PWR07
 U 1 1 559D78B1
-P 2100 5200
-F 0 "#PWR07" H 2100 4950 60  0001 C CNN
-F 1 "GNDREF" H 2100 5050 60  0000 C CNN
-F 2 "" H 2100 5200 60  0000 C CNN
-F 3 "" H 2100 5200 60  0000 C CNN
-	1    2100 5200
+P 1650 5200
+F 0 "#PWR07" H 1650 4950 60  0001 C CNN
+F 1 "GNDREF" H 1650 5050 60  0000 C CNN
+F 2 "" H 1650 5200 60  0000 C CNN
+F 3 "" H 1650 5200 60  0000 C CNN
+	1    1650 5200
 	1    0    0    -1
 $EndComp
@@
 P 5200 7400
 F 0 "R3" V 5280 7400 50  0000 C CNN
-F 1 "1K" V 5200 7400 50  0000 C CNN
+F 1 "1kΩ" V 5200 7400 50  0000 C CNN
 F 2 "Resistors_SMD:R_0805_HandSoldering" V 5130 7400 30  0001 C CNN
 F 3 "" H 5200 7400 30  0000 C CNN
@@
 	3300 6150 3450 6150
 Wire Wire Line
-	3450 4400 2700 4400
-Wire Wire Line
-	2700 4400 2700 4750
-Wire Wire Line
-	3450 4000 2100 4000
-Wire Wire Line
-	2100 4000 2100 4750
-Wire Wire Line
-	2100 4600 2250 4600
-Connection ~ 2100 4600
-Wire Wire Line
-	2550 4600 2700 4600
-Connection ~ 2700 4600
-Wire Wire Line
-	2100 5050 2100 5200
-Wire Wire Line
-	2700 5050 2700 5200
+	3450 4400 3000 4400
+Wire Wire Line
+	3000 4400 3000 4800
+Wire Wire Line
+	3450 4000 1650 4000
+Wire Wire Line
+	1650 4000 1650 4800
+Wire Wire Line
+	1650 5100 1650 5200
+Wire Wire Line
+	3000 5100 3000 5200
 Wire Wire Line
 	3450 6750 3300 6750
@@
 P 3050 6850
 F 0 "C8" H 3075 6950 50  0000 L CNN
-F 1 "1uF" H 3075 6750 50  0000 L CNN
+F 1 "1µF" H 3075 6750 50  0000 L CNN
 F 2 "Capacitors_SMD:C_0805_HandSoldering" H 3050 6850 60  0001 C CNN
 F 3 "" H 3050 6850 60  0000 C CNN
@@
 F 0 "S0:0" H 11550 4450 60  0000 C CNN
 F 1 "MX1A" H 11700 4300 60  0000 C CNN
-F 2 "CHERRY_PCB_100H:CHERRY_PCB_100H" H 11700 4200 60  0001 C CNN
+F 2 "bwu-keyboard:bwu-mx1a-1u" H 11700 4200 60  0001 C CNN
 F 3 "" H 11700 4200 60  0000 C CNN
 	1    11700 4200
@@
 F 0 "S0:1" H 12300 4450 60  0000 C CNN
 F 1 "MX1A" H 12450 4300 60  0000 C CNN
-F 2 "CHERRY_PCB_100H:CHERRY_PCB_100H" H 12450 4200 60  0001 C CNN
+F 2 "bwu-keyboard:bwu-mx1a-1u" H 12450 4200 60  0001 C CNN
 F 3 "" H 12450 4200 60  0000 C CNN
 	1    12450 4200
@@
 F 0 "S0:2" H 13050 4450 60  0000 C CNN
 F 1 "MX1A" H 13200 4300 60  0000 C CNN
-F 2 "CHERRY_PCB_100H:CHERRY_PCB_100H" H 13200 4200 60  0001 C CNN
+F 2 "bwu-keyboard:bwu-mx1a-1u" H 13200 4200 60  0001 C CNN
 F 3 "" H 13200 4200 60  0000 C CNN
 	1    13200 4200
@@
 F 0 "S1:0" H 11550 5150 60  0000 C CNN
 F 1 "MX1A" H 11700 5000 60  0000 C CNN
-F 2 "CHERRY_PCB_100H:CHERRY_PCB_100H" H 11700 4900 60  0001 C CNN
+F 2 "bwu-keyboard:bwu-mx1a-1u" H 11700 4900 60  0001 C CNN
 F 3 "" H 11700 4900 60  0000 C CNN
 	1    11700 4900
@@
 	11900 4750 11900 5000
 Wire Wire Line
-	11600 5000 11400 5000
+	11400 5000 11600 5000
 $Comp
 L MX1A S1:1
@@
 F 0 "S1:1" H 12300 5150 60  0000 C CNN
 F 1 "MX1A" H 12450 5000 60  0000 C CNN
-F 2 "CHERRY_PCB_100H:CHERRY_PCB_100H" H 12450 4900 60  0001 C CNN
+F 2 "bwu-keyboard:bwu-mx1a-1u" H 12450 4900 60  0001 C CNN
 F 3 "" H 12450 4900 60  0000 C CNN
 	1    12450 4900
@@
 F 0 "S1:2" H 13050 5150 60  0000 C CNN
 F 1 "MX1A" H 13200 5000 60  0000 C CNN
-F 2 "CHERRY_PCB_100H:CHERRY_PCB_100H" H 13200 4900 60  0001 C CNN
+F 2 "bwu-keyboard:bwu-mx1a-1u" H 13200 4900 60  0001 C CNN
 F 3 "" H 13200 4900 60  0000 C CNN
 	1    13200 4900
@@
 	13400 4750 13400 5000
 Wire Wire Line
-	13100 5000 12900 5000
+	12900 5000 13100 5000
 $Comp
 L MX1A S2:1
@@
 F 0 "S2:1" H 12300 5850 60  0000 C CNN
 F 1 "MX1A" H 12450 5700 60  0000 C CNN
-F 2 "CHERRY_PCB_100H:CHERRY_PCB_100H" H 12450 5600 60  0001 C CNN
+F 2 "bwu-keyboard:bwu-mx1a-2u" H 12450 5600 60  0001 C CNN
 F 3 "" H 12450 5600 60  0000 C CNN
 	1    12450 5600
@@
 	12650 5450 12650 5700
 Wire Wire Line
-	12350 5700 12150 5700
+	12150 5700 12350 5700
 Wire Wire Line
 	11100 3800 13000 3800
@@
 	11100 5200 12250 5200
 Wire Wire Line
-	11400 5000 11400 3500
+	11400 3500 11400 5000
 Connection ~ 11400 4300
 Wire Wire Line
-	12150 5700 12150 3500
+	12150 3500 12150 5700
 Connection ~ 12150 5000
 Connection ~ 12150 4300
 Wire Wire Line
-	12900 5000 12900 3500
+	12900 3500 12900 5000
 Connection ~ 12900 4300
 Text Label 11400 3500 0    60   ~ 0
@@
 Text Label 11100 5200 0    60   ~ 0
 B2
+$Comp
+L ABM8G Y1
+U 1 1 55C0694B
+P 2350 4600
+F 0 "Y1" H 2550 4900 60  0000 C CNN
+F 1 "ABM8G" H 2350 4300 60  0000 C CNN
+F 2 "bwu-keyboard:bwu-ABM8G-16.000MHZ-4Y-T3" H 2300 4500 60  0001 C CNN
+F 3 "" H 2300 4500 60  0000 C CNN
+	1    2350 4600
+	-1   0    0    -1
+$EndComp
+Connection ~ 1650 4450
+Wire Wire Line
+	1650 4450 1850 4450
+Connection ~ 3000 4750
+Wire Wire Line
+	2850 4750 3000 4750
+Wire Wire Line
+	1850 4750 1400 4750
+Wire Wire Line
+	1400 4750 1400 5200
+Wire Wire Line
+	2850 4450 3300 4450
+Wire Wire Line
+	3300 4450 3300 5200
+$Comp
+L GNDREF #PWR014
+U 1 1 55C08875
+P 3300 5200
+F 0 "#PWR014" H 3300 4950 60  0001 C CNN
+F 1 "GNDREF" H 3300 5050 60  0000 C CNN
+F 2 "" H 3300 5200 60  0000 C CNN
+F 3 "" H 3300 5200 60  0000 C CNN
+	1    3300 5200
+	1    0    0    -1
+$EndComp
+$Comp
+L GNDREF #PWR015
+U 1 1 55C088A6
+P 1400 5200
+F 0 "#PWR015" H 1400 4950 60  0001 C CNN
+F 1 "GNDREF" H 1400 5050 60  0000 C CNN
+F 2 "" H 1400 5200 60  0000 C CNN
+F 3 "" H 1400 5200 60  0000 C CNN
+	1    1400 5200
+	1    0    0    -1
+$EndComp
 $EndSCHEMATC

Commit message: new reset switch schematic and footprint
Parts:
- removed SW1: SW_PUSH, Buttons_Switches_SMD:SW_SPST_FSMSM, symbol SW_PUSH
- added SW1: SW423CT-ND, bwu-keyboard:bwu-SW423CT-ND, symbol SW423CT-ND
Connections:
- wire segments 107 -> 106
Other:
- moved on the sheet: D0:0, D0:1, D0:2, D1:0, D1:1, D1:2, D2:1, S0:0, S0:1, S0:2, S1:0, S1:1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

Commit message: schematic cleanup
Connections:
- net labels added: AREF, D+, D-, GND, RESET, UCAP, VCC, XTAL1, XTAL2
- net labels removed: GNDREF
- wire segments 106 -> 82
Other:
- moved on the sheet: C1, C2, C3, C4, C5, C6, C7, C8, CON1, D0:0, D0:1, D0:2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

Commit message: revision submitted to dirtypcb
Parts:
- added LED1: 5060BRG4, bwu-keyboard:bwu-5060BRG4, symbol 5060BRG4
- added R4, R6: 220Ω, bwu-keyboard:bwu-resistor-0805, symbol R
- added R5: 330Ω, bwu-keyboard:bwu-resistor-0805, symbol R
- C1, C2, C3, C4, C5, C7: footprint Capacitors_SMD:C_0805_HandSoldering -> bwu-keyboard:bwu-ceramic-capacitor-0805
- C6, C8: footprint Capacitors_SMD:C_0805_HandSoldering -> bwu-keyboard:bwu-electrolyte-capacitor-0805
- R1, R2, R3: footprint Resistors_SMD:R_0805_HandSoldering -> bwu-keyboard:bwu-resistor-0805
- Y1: value ABM8G -> 16MHz
Connections:
- net labels added: C0, C1, C2, LED_B, LED_G, LED_R, R0, R1, R2
- net labels removed: B0, B1, B2, B3, B4, B5, B6, B7, C6, C7, D0, D1, D2, D3, D4, D5, D6, D7, E6, F0, F1, F4, F5, F6, F7
- wire segments 82 -> 59
Other:
- moved on the sheet: C1, C2, C3, C4, C5, C6, C7, C8, CON1, D0:0, D0:1, D0:2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

Commit message: small schematic changes
Connections:
- net labels added: XTAL+, XTAL-
- net labels removed: XTAL1, XTAL2
Changed lines of the file:
@@
 	3650 4300 3900 4300
 Text Label 3650 4300 2    60   ~ 0
-XTAL2
+XTAL+
 Text Label 5150 4600 0    60   ~ 0
-XTAL1
+XTAL-
 Text Label 6100 3850 2    60   ~ 0
-XTAL2
+XTAL+
 Text Label 6100 4250 2    60   ~ 0
-XTAL1
+XTAL-
 Text Label 5250 7300 0    60   ~ 0
 GND
