File: granite.kicad_pcb (KiCad board)
At the start: 2 copper layers, 57.2 x 58.4 mm, 29 parts, among them CON1 USB-MINI-B WM17115-ND, IC1 ATMEGA32U4, SW1 SW_PUSH, Y1 ABM8G

Commit message: schematic cleanup
Parts:
- SW1: value SW_PUSH -> SW423CT-ND; footprint Buttons_Switches_SMD:SW_SPST_FSMSM -> bwu-keyboard:bwu-SW423CT-ND
- moved C2 36.9 mm to (158.8, 152.9), turned to 270 degrees
- moved C1 23.1 mm to (173.0, 146.3)
- moved C6 18.4 mm to (159.0, 133.3), turned to 180 degrees
- moved C3 18.2 mm to (173.0, 139.4)
- moved SW1 10.8 mm to (134.9, 146.3), turned to 270 degrees
- moved R1 5.08 mm to (165.1, 116.2)
- moved R2 5.08 mm to (162.6, 116.2)
- moved Y1 2.43 mm to (145.5, 142.0)
- moved C7 2.22 mm to (173.0, 141.7)
- moved C5 2.07 mm to (150.4, 143.3), turned to 180 degrees
- moved C4 1.59 mm to (150.4, 140.5), turned to 180 degrees
Connections:
- net Net-(C1-Pad1) renamed /VCC
- net Net-(C4-Pad1) renamed /XTAL2
- net Net-(C5-Pad1) renamed /XTAL1
- net Net-(C7-Pad1) renamed /AREF
- net Net-(C8-Pad1) renamed /UCAP
- net Net-(IC1-Pad13) renamed /RESET
- net Net-(IC1-Pad3) renamed /D-
- net Net-(IC1-Pad4) renamed /D+
- C1 pad 2: GNDREF -> /GND
- C2 pad 2: GNDREF -> /GND
- C3 pad 2: GNDREF -> /GND
- C4 pad 2: GNDREF -> /GND
- C5 pad 2: GNDREF -> /GND
- C6 pad 2: GNDREF -> /GND
- C7 pad 2: GNDREF -> /GND
- C8 pad 2: GNDREF -> /GND
- CON1 pad 5: GNDREF -> /GND
- CON1 pad 6: GNDREF -> /GND
- CON1 pad 7: GNDREF -> /GND
- D0:0 pad 2: /B7 -> /F5
- D0:1 pad 2: /B6 -> /B4
- D0:2 pad 2: /B5 -> /B6
- D1:0 pad 2: /B7 -> /F5
- D1:1 pad 2: /B6 -> /B4
- D1:2 pad 2: /B5 -> /B6
- D2:1 pad 2: /B6 -> /B4
- IC1 pad 15: GNDREF -> /GND
- IC1 pad 23: GNDREF -> /GND
- IC1 pad 35: GNDREF -> /GND
- IC1 pad 43: GNDREF -> /GND
- IC1 pad 5: GNDREF -> /GND
- R3 pad 1: Net-(IC1-Pad33) -> /GND
- R3 pad 2: GNDREF -> Net-(IC1-Pad33)
- S0:0 pad 1: /B4 -> /F7
- S0:1 pad 1: /B4 -> /F7
- S0:2 pad 1: /B4 -> /F7
- S1:0 pad 1: /B3 -> /F6
- S1:1 pad 1: /B3 -> /F6
- S1:2 pad 1: /B3 -> /F6
- S2:1 pad 1: /B2 -> /B5
- SW1 pad 1: GNDREF -> Net-(SW1-Pad1)
- Y1 pad 2: GNDREF -> /GND
- Y1 pad 4: GNDREF -> /GND
Routing:
- net /F6: track 0.00 -> 108.5 mm
- net /VCC: track 0.00 -> 101.9 mm, vias 0 -> 4
- net /F7: track 0.00 -> 96.5 mm
- net /B4: track 0.00 -> 78.7 mm
- net /B6: track 0.00 -> 76.0 mm
- net /F5: track 0.00 -> 38.6 mm
- net /B5: track 0.00 -> 31.0 mm
- net /RESET: track 0.00 -> 26.6 mm, vias 0 -> 2
- net /D+: track 0.00 -> 19.4 mm
- net /D-: track 0.00 -> 19.3 mm
- net /XTAL2: track 0.00 -> 15.0 mm
- net /UCAP: track 0.00 -> 14.9 mm
- net /XTAL1: track 0.00 -> 13.5 mm
- net /GND: track 0.00 -> 13.3 mm
- net Net-(CON1-Pad2): track 0.00 -> 8.64 mm
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Other:
- outline, holes or cut-outs redrawn

Commit message: revision submitted to dirtypcb
Parts:
- added LED1: 5060BRG4, bwu-keyboard:bwu-5060BRG4, F.Cu at (150.6, 124.0)
- added R4: 220Ω, bwu-keyboard:bwu-resistor-0805, F.Cu at (160.3, 133.5)
- added R5: 330Ω, bwu-keyboard:bwu-resistor-0805, F.Cu at (158.8, 128.2)
- added R6: 220Ω, bwu-keyboard:bwu-resistor-0805, F.Cu at (157.2, 133.5)
- C1, C2, C3, C4, C5, C7: footprint Capacitors_SMD:C_0805_HandSoldering -> bwu-keyboard:bwu-ceramic-capacitor-0805
- C6, C8: footprint Capacitors_SMD:C_0805_HandSoldering -> bwu-keyboard:bwu-electrolyte-capacitor-0805
- R1, R2, R3: footprint Resistors_SMD:R_0805_HandSoldering -> bwu-keyboard:bwu-resistor-0805
- Y1: value ABM8G -> 16MHz
- moved D0:1 12.2 mm to (142.7, 116.6)
- moved C8 10.4 mm to (162.3, 133.5), turned to 90 degrees
- moved C6 8.92 mm to (150.9, 137.0)
- moved RESET 6.40 mm to (132.2, 152.1)
- moved R3 1.77 mm to (166.0, 154.2), turned to 90 degrees
- moved C1 1.68 mm to (172.7, 148.0)
- moved IC1 1.65 mm to (161.9, 143.9)
- moved C4 1.53 mm to (149.8, 141.9)
- moved C2 1.14 mm to (158.7, 154.1)
- moved Y1 0.89 mm to (145.5, 142.9)
- moved C5 0.81 mm to (149.9, 143.9)
- moved C7 0.60 mm to (172.6, 142.2)
- moved C3 0.59 mm to (172.6, 139.9)
- renumbered SW1 to RESET
Connections:
- net /B0 renamed Net-(IC1-Pad8)
- net /B4 renamed /C1
- net /B5 renamed /R2
- net /B6 renamed /C2
- net /B7 renamed Net-(IC1-Pad12)
- net /C6 renamed Net-(IC1-Pad31)
- net /C7 renamed Net-(IC1-Pad32)
- net /D0 renamed Net-(IC1-Pad18)
- net /D1 renamed Net-(IC1-Pad19)
- net /D2 renamed Net-(IC1-Pad20)
- net /D3 renamed Net-(IC1-Pad21)
- net /D4 renamed Net-(IC1-Pad25)
- net /D5 renamed Net-(IC1-Pad22)
- net /D6 renamed Net-(IC1-Pad26)
- net /D7 renamed Net-(IC1-Pad27)
- net /E6 renamed Net-(IC1-Pad1)
- net /F0 renamed Net-(IC1-Pad41)
- net /F1 renamed Net-(IC1-Pad40)
- net /F4 renamed Net-(IC1-Pad39)
- net /F5 renamed /C0
- net /F6 renamed /R1
- net /F7 renamed /R0
- net /XTAL1 renamed /XTAL-
- net /XTAL2 renamed /XTAL+
- IC1 pad 10: /B2 -> /LED_R
- IC1 pad 11: /B3 -> /LED_G
- IC1 pad 9: /B1 -> /LED_B
Routing:
- net /GND: track 13.3 -> 83.2 mm, vias 0 -> 17
- net /R1: track 108.5 -> 59.9 mm, vias 0 -> 2
- net Net-(LED1-Pad3): track 0.00 -> 16.1 mm
- net /UCAP: track 14.9 -> 3.59 mm
- net Net-(D0:1-Pad1): track 3.38 -> 14.6 mm
- net /C1: track 78.7 -> 67.7 mm
- net Net-(LED1-Pad1): track 0.00 -> 10.1 mm
- net /LED_R: track 0.00 -> 8.31 mm
- net Net-(LED1-Pad2): track 0.00 -> 7.46 mm
- net /RESET: track 26.6 -> 33.4 mm
- net /R0: track 96.5 -> 92.2 mm
- net /VCC: track 101.9 -> 106.0 mm, vias 4 -> 6
- net /LED_B: track 0.00 -> 3.66 mm
- net /LED_G: track 0.00 -> 3.64 mm
- net Net-(CON1-Pad3): track 5.37 -> 8.87 mm
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- added copper zone on B.Cu, net /GND
- added copper zone on F.Cu, net /GND
Other:
- board text added: "keyboard proto 2"

Commit message: first routing pass finished
Parts:
- removed RESET: SW423CT-ND, bwu-keyboard:bwu-SW423CT-ND
- added D0:10: D, SM0805:SOD-123, F.Cu at (119.4, 50.4)
- added D0:11: D, SM0805:SOD-123, F.Cu at (100.3, 50.4)
- added D0:12: D, SM0805:SOD-123, F.Cu at (81.3, 50.4)
- added D0:13: D, SM0805:SOD-123, F.Cu at (57.5, 50.4)
- added D0:3: D, SM0805:SOD-123, F.Cu at (252.7, 50.4)
- added D0:4: D, SM0805:SOD-123, F.Cu at (233.7, 50.4)
- added D0:5: D, SM0805:SOD-123, F.Cu at (214.6, 50.4)
- added D0:6: D, SM0805:SOD-123, F.Cu at (195.6, 50.4)
- added D0:7: D, SM0805:SOD-123, F.Cu at (176.5, 50.4)
- added D0:8: D, SM0805:SOD-123, F.Cu at (157.5, 50.4)
- added D0:9: D, SM0805:SOD-123, F.Cu at (138.4, 50.4)
- added D1:10: D, SM0805:SOD-123, F.Cu at (119.4, 69.4)
- added D1:11: D, SM0805:SOD-123, F.Cu at (100.3, 69.4)
- added D1:12: D, SM0805:SOD-123, F.Cu at (81.3, 69.4)
- added D1:13: D, SM0805:SOD-123, F.Cu at (57.5, 69.4)
- added D1:3: D, SM0805:SOD-123, F.Cu at (252.7, 69.4)
- added D1:4: D, SM0805:SOD-123, F.Cu at (233.7, 69.4)
- added D1:5: D, SM0805:SOD-123, F.Cu at (214.6, 69.4)
- added D1:6: D, SM0805:SOD-123, F.Cu at (195.6, 69.4)
- added D1:7: D, SM0805:SOD-123, F.Cu at (167.3, 65.2)
- added D1:8: D, SM0805:SOD-123, F.Cu at (157.5, 69.4)
- added D1:9: D, SM0805:SOD-123, F.Cu at (138.4, 69.4)
- added D2:0: D, SM0805:SOD-123, F.Cu at (315.0, 88.5)
- added D2:10: D, SM0805:SOD-123, F.Cu at (119.4, 88.1)
- added D2:11: D, SM0805:SOD-123, F.Cu at (100.3, 88.1)
- added D2:12: D, SM0805:SOD-123, F.Cu at (81.3, 88.5)
- added D2:13: D, SM0805:SOD-123, F.Cu at (57.5, 88.5)
- added D2:2: D, SM0805:SOD-123, F.Cu at (271.8, 88.5)
- added D2:3: D, SM0805:SOD-123, F.Cu at (252.7, 88.5)
- added D2:4: D, SM0805:SOD-123, F.Cu at (233.7, 88.5)
- added D2:5: D, SM0805:SOD-123, F.Cu at (214.6, 88.5)
- added D2:6: D, SM0805:SOD-123, F.Cu at (188.3, 84.2)
- added D2:7: D, SM0805:SOD-123, F.Cu at (176.5, 88.5)
- added D2:8: D, SM0805:SOD-123, F.Cu at (157.5, 88.5)
- added D2:9: D, SM0805:SOD-123, F.Cu at (138.4, 88.5)
- added D3:0: D, SM0805:SOD-123, F.Cu at (315.0, 107.5)
- added D3:1: D, SM0805:SOD-123, F.Cu at (290.8, 107.5)
- added D3:10: D, SM0805:SOD-123, F.Cu at (119.4, 107.5)
- added D3:11: D, SM0805:SOD-123, F.Cu at (100.3, 107.5)
- added D3:12: D, SM0805:SOD-123, F.Cu at (81.3, 107.5)
- added D3:13: D, SM0805:SOD-123, F.Cu at (57.5, 107.5)
- added D3:2: D, SM0805:SOD-123, F.Cu at (271.8, 107.5)
- added D3:3: D, SM0805:SOD-123, F.Cu at (252.7, 107.5)
- added D3:4: D, SM0805:SOD-123, F.Cu at (233.7, 107.5)
- added D3:5: D, SM0805:SOD-123, F.Cu at (214.6, 107.5)
- added D3:6: D, SM0805:SOD-123, F.Cu at (195.6, 107.5)
- added D3:7: D, SM0805:SOD-123, F.Cu at (176.5, 107.5)
- added D3:8: D, SM0805:SOD-123, F.Cu at (157.5, 107.5)
- added D3:9: D, SM0805:SOD-123, F.Cu at (138.4, 107.5)
- added D4:0: D, SM0805:SOD-123, F.Cu at (317.5, 126.6)
- added D4:1: D, SM0805:SOD-123, F.Cu at (293.4, 126.6)
- added D4:10: D, SM0805:SOD-123, F.Cu at (127.0, 126.6)
- added D4:11: D, SM0805:SOD-123, F.Cu at (102.9, 126.6)
- added D4:12: D, SM0805:SOD-123, F.Cu at (78.7, 126.6)
- added D4:13: D, SM0805:SOD-123, F.Cu at (55.1, 126.6)
- added D4:2: D, SM0805:SOD-123, F.Cu at (269.2, 126.6)
- added D4:3: D, SM0805:SOD-123, F.Cu at (245.1, 126.6)
- added D4:5: D, SM0805:SOD-123, F.Cu at (219.7, 126.6)
- added D4:6: D, SM0805:SOD-123, F.Cu at (177.3, 122.3)
- added D4:8: D, SM0805:SOD-123, F.Cu at (152.4, 126.6)
- added LED2: 5060BRG4, bwu-keyboard:bwu-5060BRG4, F.Cu at (106.1, 93.7)
- added LED3: 5060BRG4, bwu-keyboard:bwu-5060BRG4, F.Cu at (144.2, 93.7)
- added LED4: 5060BRG4, bwu-keyboard:bwu-5060BRG4, F.Cu at (182.3, 93.7)
- added LED5: 5060BRG4, bwu-keyboard:bwu-5060BRG4, F.Cu at (220.4, 93.7)
- added LED6: 5060BRG4, bwu-keyboard:bwu-5060BRG4, F.Cu at (258.5, 93.7)
- added LED7: 5060BRG4, bwu-keyboard:bwu-5060BRG4, F.Cu at (296.6, 93.7)
- added Q1: NMOSFET, bwu-keyboard:IRLML2502, F.Cu at (45.5, 97.8)
- added Q2: NMOSFET, bwu-keyboard:IRLML2502, F.Cu at (45.5, 93.7)
- added Q3: NMOSFET, bwu-keyboard:IRLML2502, F.Cu at (45.5, 89.7)
- added R10: 220Ω, bwu-keyboard:bwu-resistor-0805, F.Cu at (160.7, 83.3)
- added R11: 330Ω, bwu-keyboard:bwu-resistor-0805, F.Cu at (163.2, 83.3)
- added R12: 220Ω, bwu-keyboard:bwu-resistor-0805, F.Cu at (165.7, 83.3)
- added R13: 220Ω, bwu-keyboard:bwu-resistor-0805, F.Cu at (198.8, 83.3)
- added R14: 330Ω, bwu-keyboard:bwu-resistor-0805, F.Cu at (201.3, 83.3)
- added R15: 220Ω, bwu-keyboard:bwu-resistor-0805, F.Cu at (203.8, 83.3)
- added R16: 220Ω, bwu-keyboard:bwu-resistor-0805, F.Cu at (236.9, 83.3)
- added R17: 330Ω, bwu-keyboard:bwu-resistor-0805, F.Cu at (239.4, 83.3)
- added R18: 220Ω, bwu-keyboard:bwu-resistor-0805, F.Cu at (241.9, 83.3)
- added R19: 220Ω, bwu-keyboard:bwu-resistor-0805, F.Cu at (275.0, 83.3)
- added R20: 330Ω, bwu-keyboard:bwu-resistor-0805, F.Cu at (277.5, 83.3)
- added R21: 220Ω, bwu-keyboard:bwu-resistor-0805, F.Cu at (280.0, 83.3)
- added R22: 220Ω, bwu-keyboard:bwu-resistor-0805, F.Cu at (317.0, 83.3)
- added R23: 330Ω, bwu-keyboard:bwu-resistor-0805, F.Cu at (319.5, 83.3)
- added R24: 220Ω, bwu-keyboard:bwu-resistor-0805, F.Cu at (322.1, 83.3)
- added R25: 1kΩ, bwu-keyboard:bwu-resistor-0805, F.Cu at (57.3, 97.1)
- added R26: 1kΩ, bwu-keyboard:bwu-resistor-0805, F.Cu at (49.5, 95.8)
- added R27: 1kΩ, bwu-keyboard:bwu-resistor-0805, F.Cu at (49.5, 91.6)
- added R7: 220Ω, bwu-keyboard:bwu-resistor-0805, F.Cu at (122.6, 83.3)
- added R8: 330Ω, bwu-keyboard:bwu-resistor-0805, F.Cu at (125.1, 83.3)
- added R9: 220Ω, bwu-keyboard:bwu-resistor-0805, F.Cu at (127.6, 83.3)
- added S0:10: K_8, bwu-keyboard:bwu-mx1a-1u, B.Cu at (115.6, 47.0)
- added S0:11: K_9, bwu-keyboard:bwu-mx1a-1u, B.Cu at (96.5, 47.0)
- added S0:12: K_0, bwu-keyboard:bwu-mx1a-1u, B.Cu at (77.5, 47.0)
- added S0:13: K_EQUAL, bwu-keyboard:bwu-mx1a-150u, B.Cu at (53.7, 47.0)
- added S0:3: K_3, bwu-keyboard:bwu-mx1a-1u, B.Cu at (248.9, 47.0)
- added S0:4: K_4, bwu-keyboard:bwu-mx1a-1u, B.Cu at (229.9, 47.0)
- added S0:5: K_5, bwu-keyboard:bwu-mx1a-1u, B.Cu at (210.8, 47.0)
- added S0:6: K_BL1, bwu-keyboard:bwu-mx1a-1u, B.Cu at (191.8, 47.0)
- added S0:7: K_BL2, bwu-keyboard:bwu-mx1a-1u, B.Cu at (172.7, 47.0)
- added S0:8: K_6, bwu-keyboard:bwu-mx1a-1u, B.Cu at (153.7, 47.0)
- added S0:9: K_7, bwu-keyboard:bwu-mx1a-1u, B.Cu at (134.6, 47.0)
- added S1:10: K_C, bwu-keyboard:bwu-mx1a-1u, B.Cu at (115.6, 66.0)
- added S1:11: K_R, bwu-keyboard:bwu-mx1a-1u, B.Cu at (96.5, 66.0)
- added S1:12: K_L, bwu-keyboard:bwu-mx1a-1u, B.Cu at (77.5, 66.0)
- added S1:13: K_SLASH, bwu-keyboard:bwu-mx1a-150u, B.Cu at (53.7, 66.0)
- added S1:3: K_PRD, bwu-keyboard:bwu-mx1a-1u, B.Cu at (248.9, 66.0)
- added S1:4: K_P, bwu-keyboard:bwu-mx1a-1u, B.Cu at (229.9, 66.0)
- added S1:5: K_Y, bwu-keyboard:bwu-mx1a-1u, B.Cu at (210.8, 66.0)
- added S1:6: K_HOME, bwu-keyboard:bwu-mx1a-1u, B.Cu at (191.8, 66.0)
- added S1:7: K_PGUP, bwu-keyboard:bwu-mx1a-1u, B.Cu at (172.7, 66.0)
- added S1:8: K_F, bwu-keyboard:bwu-mx1a-1u, B.Cu at (153.7, 66.0)
- added S1:9: K_G, bwu-keyboard:bwu-mx1a-1u, B.Cu at (134.6, 66.0)
- added S2:0: K_BKTK, bwu-keyboard:bwu-mx1a-150u, B.Cu at (310.8, 85.1)
- added S2:10: K_T, bwu-keyboard:bwu-mx1a-1u, B.Cu at (115.6, 85.1)
- added S2:11: K_N, bwu-keyboard:bwu-mx1a-1u, B.Cu at (96.5, 85.1)
- added S2:12: K_S, bwu-keyboard:bwu-mx1a-1u, B.Cu at (77.5, 85.1)
- added S2:13: K_DASH, bwu-keyboard:bwu-mx1a-150u, B.Cu at (53.7, 85.1)
- added S2:2: K_O, bwu-keyboard:bwu-mx1a-1u, B.Cu at (268.0, 85.1)
- added S2:3: K_E, bwu-keyboard:bwu-mx1a-1u, B.Cu at (248.9, 85.1)
- added S2:4: K_U, bwu-keyboard:bwu-mx1a-1u, B.Cu at (229.9, 85.1)
- added S2:5: K_I, bwu-keyboard:bwu-mx1a-1u, B.Cu at (210.8, 85.1)
- added S2:6: K_END, bwu-keyboard:bwu-mx1a-1u, B.Cu at (191.8, 85.1)
- added S2:7: K_PGDN, bwu-keyboard:bwu-mx1a-1u, B.Cu at (172.7, 85.1)
- added S2:8: K_D, bwu-keyboard:bwu-mx1a-1u, B.Cu at (153.7, 85.1)
- added S2:9: K_H, bwu-keyboard:bwu-mx1a-1u, B.Cu at (134.6, 85.1)
- added S3:0: K_LSHFT, bwu-keyboard:bwu-mx1a-150u, B.Cu at (310.8, 104.1)
- added S3:1: K_SMCLN, bwu-keyboard:bwu-mx1a-1u, B.Cu at (287.0, 104.1)
- added S3:10: K_W, bwu-keyboard:bwu-mx1a-1u, B.Cu at (115.6, 104.1)
- added S3:11: K_V, bwu-keyboard:bwu-mx1a-1u, B.Cu at (96.5, 104.1)
- added S3:12: K_Z, bwu-keyboard:bwu-mx1a-1u, B.Cu at (77.5, 104.1)
- added S3:13: K_RSHFT, bwu-keyboard:bwu-mx1a-150u, B.Cu at (53.7, 104.1)
- added S3:2: K_Q, bwu-keyboard:bwu-mx1a-1u, B.Cu at (268.0, 104.1)
- added S3:3: K_J, bwu-keyboard:bwu-mx1a-1u, B.Cu at (248.9, 104.1)
- added S3:4: K_K, bwu-keyboard:bwu-mx1a-1u, B.Cu at (229.9, 104.1)
- added S3:5: K_X, bwu-keyboard:bwu-mx1a-1u, B.Cu at (210.8, 104.1)
- added S3:6: K_DEL, bwu-keyboard:bwu-mx1a-1u, B.Cu at (191.8, 104.1)
- added S3:7: K_INS, bwu-keyboard:bwu-mx1a-1u, B.Cu at (172.7, 104.1)
- added S3:8: K_B, bwu-keyboard:bwu-mx1a-1u, B.Cu at (153.7, 104.1)
- added S3:9: K_M, bwu-keyboard:bwu-mx1a-1u, B.Cu at (134.6, 104.1)
- added S4:0: K_LCTRL, bwu-keyboard:bwu-mx1a-125u, B.Cu at (313.2, 123.2)
- added S4:1: K_LGUI, bwu-keyboard:bwu-mx1a-125u, B.Cu at (289.4, 123.2)
- added S4:10: K_RFN, bwu-keyboard:bwu-mx1a-125u, B.Cu at (122.7, 123.2)
- added S4:11: K_RALT, bwu-keyboard:bwu-mx1a-125u, B.Cu at (98.9, 123.2)
- added S4:12: K_RGUI, bwu-keyboard:bwu-mx1a-125u, B.Cu at (75.1, 123.2)
- added S4:13: K_RCTRL, bwu-keyboard:bwu-mx1a-125u, B.Cu at (51.3, 123.2)
- added S4:2: K_LALT, bwu-keyboard:bwu-mx1a-125u, B.Cu at (265.6, 123.2)
- added S4:3: K_LFN, bwu-keyboard:bwu-mx1a-125u, B.Cu at (241.8, 123.2)
- added S4:5: K_BKSPC, bwu-keyboard:bwu-mx1a-150u, B.Cu at (215.6, 123.2)
- added S4:6: K_SPACE, bwu-keyboard:bwu-mx1a-2u, B.Cu at (182.2, 123.2)
- added S4:8: K_ENTER, bwu-keyboard:bwu-mx1a-150u, B.Cu at (148.9, 123.2)
- added SW1: SW423CT-ND, bwu-keyboard:bwu-SW423CT-ND, F.Cu at (163.2, 46.2)
- S0:0: value MX1A -> K_ESC; footprint bwu-keyboard:bwu-mx1a-1u -> bwu-keyboard:bwu-mx1a-150u
- S0:1: value MX1A -> K_1
- S0:2: value MX1A -> K_2
- S1:0: value MX1A -> K_TAB; footprint bwu-keyboard:bwu-mx1a-1u -> bwu-keyboard:bwu-mx1a-150u
- S1:1: value MX1A -> K_QUOTE
- S1:2: value MX1A -> K_COMMA
- S2:1: value MX1A -> K_A; footprint bwu-keyboard:bwu-mx1a-2u -> bwu-keyboard:bwu-mx1a-1u
- moved D0:1 162.2 mm to (290.8, 50.4)
- moved D1:1 156.8 mm to (290.8, 69.4)
- moved S0:0 155.9 mm to (310.8, 47.0)
- moved S1:0 155.9 mm to (310.8, 66.0)
- moved D0:0 155.9 mm to (315.0, 50.4)
- moved D1:0 155.9 mm to (315.0, 69.4)
- moved S0:1 151.6 mm to (287.0, 47.0)
- moved S0:2 151.6 mm to (268.0, 47.0)
- moved S1:2 151.6 mm to (268.0, 66.0)
- moved S2:1 151.6 mm to (287.0, 85.1)
- moved S1:1 151.6 mm to (287.0, 66.0)
- moved D0:2 151.3 mm to (271.8, 50.4)
- moved D1:2 151.3 mm to (271.8, 69.4)
- moved D2:1 151.2 mm to (290.8, 88.7)
- moved C2 92.8 mm to (188.5, 66.1), turned to 90 degrees
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Connections:
- net Net-(CON1-Pad2) renamed /USB_D-
- net Net-(CON1-Pad3) renamed /USB_D+
- IC1 pad 1: Net-(IC1-Pad1) -> /R1
- IC1 pad 10: /LED_R -> /LED_R_CTL
- IC1 pad 11: /LED_G -> /LED_G_CTL
- IC1 pad 12: Net-(IC1-Pad12) -> /CA
- IC1 pad 18: Net-(IC1-Pad18) -> /CD
- IC1 pad 19: Net-(IC1-Pad19) -> /CC
- IC1 pad 20: Net-(IC1-Pad20) -> /CB
- IC1 pad 21: Net-(IC1-Pad21) -> /C9
- IC1 pad 22: Net-(IC1-Pad22) -> /R3
- IC1 pad 25: Net-(IC1-Pad25) -> /C7
- IC1 pad 26: Net-(IC1-Pad26) -> /R4
- IC1 pad 27: Net-(IC1-Pad27) -> /C6
- IC1 pad 28: /C1 -> /C5
- IC1 pad 29: /R2 -> /C4
- IC1 pad 30: /C2 -> /C3
- IC1 pad 31: Net-(IC1-Pad31) -> /C2
- IC1 pad 32: Net-(IC1-Pad32) -> /C1
- IC1 pad 36: /R0 -> /R2
- IC1 pad 37: /R1 -> /C0
- IC1 pad 38: /C0 -> /R0
- IC1 pad 8: Net-(IC1-Pad8) -> /C8
- IC1 pad 9: /LED_B -> /LED_B_CTL
- LED1 pad 4: /GND -> /LED_B_Q
- LED1 pad 5: /GND -> /LED_R_Q
- LED1 pad 6: /GND -> /LED_G_Q
- R4 pad 1: /LED_B -> Net-(LED1-Pad3)
- R4 pad 2: Net-(LED1-Pad3) -> /VCC
- R5 pad 1: /LED_R -> Net-(LED1-Pad2)
- R5 pad 2: Net-(LED1-Pad2) -> /VCC
- R6 pad 1: /LED_G -> Net-(LED1-Pad1)
- R6 pad 2: Net-(LED1-Pad1) -> /VCC
Routing:
- net /VCC: track 106.0 -> 474.0 mm, vias 6 -> 3
- net /LED_G_Q: track 0.00 -> 304.3 mm, vias 0 -> 2
- net /R4: track 0.00 -> 302.6 mm
- net /R3: track 0.00 -> 297.1 mm
- net /LED_R_Q: track 0.00 -> 295.2 mm, vias 0 -> 2
- net /LED_B_Q: track 0.00 -> 288.5 mm, vias 0 -> 2
- net /R2: track 32.9 -> 266.9 mm, vias 1 -> 0
- net /CD: track 0.00 -> 229.2 mm, vias 0 -> 5
- net /R0: track 92.2 -> 304.6 mm, vias 0 -> 2
- net /C0: track 39.3 -> 245.7 mm, vias 0 -> 5
- net /R1: track 59.9 -> 265.1 mm, vias 2 -> 0
- net /CC: track 0.00 -> 193.4 mm, vias 0 -> 5
- net /C3: track 0.00 -> 189.7 mm, vias 0 -> 5
- net /LED_B_CTL: track 0.00 -> 179.4 mm
- net /CB: track 0.00 -> 175.7 mm, vias 0 -> 7
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- removed copper zone on F.Cu, net /GND
Other:
- board size 57.2 x 58.4 mm -> 285.8 x 97.2 mm
- board text removed: "keyboard proto 2"

Commit message: replacing mosfets with dedicated led driver chip
Parts:
- removed Q1, Q2, Q3: NMOSFET, bwu-keyboard:IRLML2502
- removed R10, R12, R13, R15, R16, R18, R19, R21, R22, R24, R9: 220Ω, bwu-keyboard:bwu-resistor-0805
- removed R11, R14, R17, R20, R23: 330Ω, bwu-keyboard:bwu-resistor-0805
- removed R25, R26, R27: 1kΩ, bwu-keyboard:bwu-resistor-0805
- added C10: 100nF, bwu-keyboard:bwu-ceramic-capacitor-0805, F.Cu at (206.8, 84.3)
- added C9: 220nF, bwu-keyboard:bwu-ceramic-capacitor-0805, F.Cu at (204.0, 84.3)
- added IC2: IS31FL3731, bwu-keyboard:SSOP-28, F.Cu at (202.2, 76.3)
- R4, R6: value 220Ω -> 4.7kΩ
- R5: value 330Ω -> 4.7kΩ
- R7: value 220Ω -> 100kΩ
- R8: value 330Ω -> 20kΩ
- moved R4 128.3 mm to (212.6, 78.2), turned to 0 degrees
- moved R5 125.8 mm to (212.6, 75.9), turned to 180 degrees
- moved R6 116.9 mm to (205.5, 68.3)
- moved R7 82.1 mm to (203.3, 68.3), turned to 270 degrees
- moved R8 73.4 mm to (198.5, 84.5)
- moved D1:6 2.19 mm to (195.6, 67.2)
- moved C7 1.53 mm to (192.0, 69.5)
Connections:
- IC1 pad 10: /LED_R_CTL -> Net-(IC1-Pad10)
- IC1 pad 11: /LED_G_CTL -> Net-(IC1-Pad11)
- IC1 pad 38: /R0 -> /SDA
- IC1 pad 39: Net-(IC1-Pad39) -> /SCL
- IC1 pad 40: Net-(IC1-Pad40) -> /INTB
- IC1 pad 41: Net-(IC1-Pad41) -> /SDB
- IC1 pad 8: /C8 -> /R0
- IC1 pad 9: /LED_B_CTL -> /C8
- LED1 pad 1: Net-(LED1-Pad1) -> /CA1
- LED1 pad 2: Net-(LED1-Pad2) -> /CA1
- LED1 pad 3: Net-(LED1-Pad3) -> /CA2
- LED1 pad 4: /LED_B_Q -> /CA1
- LED1 pad 5: /LED_R_Q -> /CA2
- LED1 pad 6: /LED_G_Q -> /CA3
- LED2 pad 1: Net-(LED2-Pad1) -> /CA2
- LED2 pad 2: Net-(LED2-Pad2) -> /CA3
- LED2 pad 3: Net-(LED2-Pad3) -> /CA3
- LED2 pad 4: /LED_B_Q -> /CA1
- LED2 pad 5: /LED_R_Q -> /CA2
- LED2 pad 6: /LED_G_Q -> /CA3
- LED3 pad 1: Net-(LED3-Pad1) -> /CA4
- LED3 pad 2: Net-(LED3-Pad2) -> /CA4
- LED3 pad 3: Net-(LED3-Pad3) -> /CA4
- LED3 pad 4: /LED_B_Q -> /CA1
- LED3 pad 5: /LED_R_Q -> /CA2
- LED3 pad 6: /LED_G_Q -> /CA3
- LED4 pad 1: Net-(LED4-Pad1) -> /CA5
- LED4 pad 2: Net-(LED4-Pad2) -> /CA5
- LED4 pad 3: Net-(LED4-Pad3) -> /CA5
- LED4 pad 4: /LED_B_Q -> /CA1
- LED4 pad 5: /LED_R_Q -> /CA2
- LED4 pad 6: /LED_G_Q -> /CA3
- LED5 pad 1: Net-(LED5-Pad1) -> /CA6
- LED5 pad 2: Net-(LED5-Pad2) -> /CA6
- LED5 pad 3: Net-(LED5-Pad3) -> /CA6
- LED5 pad 4: /LED_B_Q -> /CA1
- LED5 pad 5: /LED_R_Q -> /CA2
- LED5 pad 6: /LED_G_Q -> /CA3
- LED6 pad 1: Net-(LED6-Pad1) -> /CA7
- LED6 pad 2: Net-(LED6-Pad2) -> /CA7
- LED6 pad 3: Net-(LED6-Pad3) -> /CA7
- LED6 pad 4: /LED_B_Q -> /CA1
- LED6 pad 5: /LED_R_Q -> /CA2
- LED6 pad 6: /LED_G_Q -> /CA3
- LED7 pad 1: Net-(LED7-Pad1) -> /CA8
- LED7 pad 2: Net-(LED7-Pad2) -> /CA8
- LED7 pad 3: Net-(LED7-Pad3) -> /CA8
- LED7 pad 4: /LED_B_Q -> /CA1
- LED7 pad 5: /LED_R_Q -> /CA2
- LED7 pad 6: /LED_G_Q -> /CA3
- R4 pad 1: Net-(LED1-Pad3) -> /SDA
- R5 pad 1: Net-(LED1-Pad2) -> /VCC
- R5 pad 2: /VCC -> /SCL
- R6 pad 1: Net-(LED1-Pad1) -> /INTB
- R7 pad 1: Net-(LED2-Pad3) -> /GND
- R7 pad 2: /VCC -> /SDB
- R8 pad 1: Net-(LED2-Pad2) -> /GND
- R8 pad 2: /VCC -> Net-(IC2-Pad6)
Routing:
- net /LED_G_Q: track 304.3 -> 0.00 mm, vias 2 -> 0
- net /LED_R_Q: track 295.2 -> 0.00 mm, vias 2 -> 0
- net /LED_B_Q: track 288.5 -> 0.00 mm, vias 2 -> 0
- net /CA3: track 0.00 -> 274.3 mm, vias 0 -> 5
- net /CA1: track 0.00 -> 268.9 mm, vias 0 -> 5
- net /CA2: track 0.00 -> 263.8 mm, vias 0 -> 11
- net /VCC: track 474.0 -> 224.6 mm, vias 3 -> 4
- net /LED_B_CTL: track 179.4 -> 0.00 mm
- net /LED_R_CTL: track 173.3 -> 0.00 mm
- net /LED_G_CTL: track 167.6 -> 0.00 mm
- net /CA8: track 0.00 -> 113.9 mm
- net /CA7: track 0.00 -> 75.6 mm
- net /CA4: track 0.00 -> 70.5 mm, vias 0 -> 2
- net /CA6: track 0.00 -> 46.1 mm
- net /CA5: track 0.00 -> 38.2 mm
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
Commit message: adding ground fill to front side of pcb
Routing:
- added copper zone on F.Cu, net /GND

Commit message: some routing cleanup
Parts:
- moved D4:10 0.48 mm to (126.5, 126.6)
- moved D2:9 0.41 mm to (138.4, 88.1)
- moved D4:12 0.16 mm to (78.9, 126.6)
- moved D4:11 0.16 mm to (102.7, 126.6)
Connections:
- IC1 pad 12: /CA -> /C9
- IC1 pad 18: /CD -> /CA
- IC1 pad 19: /CC -> /CB
- IC1 pad 20: /CB -> /CC
- IC1 pad 21: /C9 -> /CD
Routing:
- net /VCC: track 224.6 -> 174.9 mm
- net /RESET: track 69.0 -> 30.6 mm
- net /CD: track 229.2 -> 219.8 mm, vias 5 -> 2
- net /C8: track 156.2 -> 148.4 mm, vias 6 -> 2
- net /CB: track 175.7 -> 169.9 mm, vias 7 -> 4
- net /C5: track 148.0 -> 142.8 mm
- net /CC: track 193.4 -> 197.4 mm, vias 5 -> 4
- net /GND: track 91.2 -> 87.9 mm, vias 18 -> 17
- net /CA: track 159.4 -> 156.8 mm
- net /R3: track 297.1 -> 296.1 mm
- net /C9: track 109.9 -> 109.6 mm, vias 7 -> 4

Commit message: hermes rev. 1
Parts:
- added REF**: benzene, bwu-keyboard:benzene, F.Cu at (195.6, 118.1)
- moved D4:6 9.73 mm to (186.1, 126.6)
- moved R4 1.11 mm to (212.6, 77.1)
- moved R5 1.11 mm to (212.6, 74.8)
- moved D4:0 0.48 mm to (317.0, 126.6)
- moved D4:3 0.48 mm to (245.6, 126.6)
- moved D0:0 0.32 mm to (314.6, 50.4)
- moved D1:0 0.32 mm to (314.6, 69.4)
- moved D2:0 0.32 mm to (314.6, 88.5)
- moved D3:0 0.32 mm to (314.6, 107.5)
- moved D4:5 0.32 mm to (219.4, 126.6)
- moved D4:8 0.32 mm to (152.7, 126.6)
- moved D4:1 0.16 mm to (293.2, 126.6)
- moved D4:2 0.16 mm to (269.4, 126.6)
Routing:
- net /GND: track 87.9 -> 125.5 mm, vias 17 -> 15
- net /R3: track 296.1 -> 282.9 mm, vias 0 -> 1
- net /C3: track 189.7 -> 195.5 mm
- net /C2: track 198.1 -> 203.2 mm
- net Net-(D4:6-Pad1): track 8.76 -> 4.22 mm
- net /R2: track 266.9 -> 270.5 mm, vias 0 -> 1
- net /CA3: track 274.3 -> 276.7 mm
- net /CA2: track 263.8 -> 266.1 mm
- net /C7: track 132.6 -> 130.9 mm
- net /CA6: track 46.1 -> 44.4 mm, vias 0 -> 2
- net /C5: track 142.8 -> 141.4 mm
- net /SDA: track 27.6 -> 29.0 mm
- net /VCC: track 174.9 -> 173.7 mm
- net /C1: track 222.5 -> 223.6 mm
- net /C6: track 120.7 -> 121.6 mm
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Other:
- outline, holes or cut-outs redrawn
- board text added: "Hermes rev. 1"
