File: hermes.sch (KiCad schematic (older format))
At the start: 164 parts, among them CON1 USB-MINI-B WM17115-ND, IC1 ATMEGA32U4, IC2 IS31FL3731, SW1 SW423CT-ND, Y1 16MHz

Commit message: library cleanup
Parts:
- IC1: footprint tqfp:TQFP44 -> bwu-keyboard:TQFP44
Changed lines of the file:
@@
 EESchema Schematic File Version 2
 LIBS:keyboard-bwu
-LIBS:power
-LIBS:device
-LIBS:transistors
-LIBS:conn
-LIBS:linear
-LIBS:regul
-LIBS:74xx
-LIBS:cmos4000
-LIBS:adc-dac
-LIBS:memory
-LIBS:xilinx
-LIBS:special
-LIBS:microcontrollers
-LIBS:dsp
-LIBS:microchip
-LIBS:analog_switches
-LIBS:motorola
-LIBS:texas
-LIBS:intel
-LIBS:audio
-LIBS:interface
-LIBS:digital-audio
-LIBS:philips
-LIBS:display
-LIBS:cypress
-LIBS:siliconi
-LIBS:opto
-LIBS:atmel
-LIBS:contrib
-LIBS:valves
-LIBS:atmega
-LIBS:mx1a
-LIBS:usb-b
-LIBS:hermes-cache
 EELAYER 25 0
 EELAYER END
@@
 F 0 "IC1" H 2150 6980 50  0000 L BNN
 F 1 "ATMEGA32U4" H 3200 3250 50  0000 L BNN
-F 2 "tqfp:TQFP44" H 3450 3175 50  0001 C CNN
+F 2 "bwu-keyboard:TQFP44" H 3450 3175 50  0001 C CNN
 F 3 "" H 2950 5150 60  0000 C CNN
 	1    2950 5150
