File: hermes.sch (KiCad schematic (older format))
At the start: 164 parts, among them CON1 USB-MINI-B WM17115-ND, IC1 ATMEGA32U4, IC2 IS31FL3731, SW1 SW423CT-ND, Y1 16MHz

Commit message: library cleanup (SOD123)
Parts:
- D0:0, D0:1, D0:10, D0:11, D0:12, D0:13, D0:2, D0:3, D0:4, D0:5, D0:6, D0:7, D0:8, D0:9, D1:0, D1:1, D1:10, D1:11, D1:12, D1:13, D1:2, D1:3, D1:4, D1:5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: footprint SM0805:SOD-123 -> bwu-keyboard:SOD-123
