File: aphrodite/aphrodite.kicad_pcb (KiCad board)
At the start: 2 copper layers, 381 x 127.8 mm, 191 parts, among them CON1 USB-MINI-B WM17115-ND, IC1 ATMEGA32U4, SW1 SW423CT-ND, Y1 16MHz

Commit message: first pass on aphrodite routing
Parts:
- moved R3 6.61 mm to (233.2, 114.5), turned to 180 degrees
- moved SW1 5.81 mm to (184.9, 43.0)
- moved C7 3.57 mm to (230.6, 103.2)
Connections:
- IC1 pad 25: /R3 -> Net-(IC1-Pad25)
- IC1 pad 28: /C5 -> /C0
- IC1 pad 29: /C4 -> /C1
- IC1 pad 30: /C3 -> /C2
- IC1 pad 31: /C2 -> /C3
- IC1 pad 32: /C1 -> /C4
- IC1 pad 36: /R2 -> /C5
- IC1 pad 37: /C0 -> /R0
- IC1 pad 38: /R0 -> /C6
- IC1 pad 39: Net-(IC1-Pad39) -> /C7
- IC1 pad 40: Net-(IC1-Pad40) -> /R3
- IC1 pad 41: Net-(IC1-Pad41) -> /R2
- IC1 pad 8: /C6 -> Net-(IC1-Pad8)
- IC1 pad 9: /C7 -> Net-(IC1-Pad9)
Routing:
- net /C0: track 131.9 -> 356.9 mm
- net /C1: track 133.3 -> 340.2 mm, vias 0 -> 2
- net /C2: track 131.0 -> 317.6 mm, vias 0 -> 2
- net /C3: track 102.9 -> 269.3 mm, vias 0 -> 2
- net /C4: track 124.4 -> 270.6 mm, vias 0 -> 2
- net /C7: track 160.6 -> 291.1 mm, vias 4 -> 2
- net /R0: track 366.0 -> 493.4 mm
- net /C5: track 103.2 -> 222.1 mm, vias 0 -> 2
- net /RESET: track 0.00 -> 74.9 mm, vias 0 -> 2
- net /R2: track 372.3 -> 425.4 mm, vias 0 -> 2
- net /R1: track 356.9 -> 395.4 mm, vias 0 -> 2
- net /GND: track 34.7 -> 67.0 mm, vias 4 -> 11
- net /R3: track 451.0 -> 421.0 mm, vias 0 -> 3
- net /C9: track 211.6 -> 238.9 mm
- net /C6: track 193.2 -> 210.8 mm
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- added copper zone on B.Cu, net /GND
- added copper zone on F.Cu, net /GND
Other:
- outline, holes or cut-outs redrawn
