File: gaia/gaia.kicad_pcb (KiCad board)
At the start: 2 copper layers, 103 parts, among them CON1 USB-MINI-B WM17115-ND, IC1 ATMEGA32U4, IC2 IS31FL3731, IC3 IS31FL3731, IC4 IS31FL3731, SW1 SW423CT-ND, Y1 16MHz

Commit message: routing
Parts:
- moved IC4 42.5 mm to (260.0, 169.4)
- moved R6 42.4 mm to (244.1, 263.0)
- moved S3:10 42.4 mm to (353.7, 132.9)
- moved S3:3 42.4 mm to (163.2, 132.9)
- moved S4:5 42.4 mm to (201.3, 156.7)
- moved S4:6 42.4 mm to (222.7, 156.7)
- moved S4:7 42.4 mm to (294.1, 156.7)
- moved S4:8 42.4 mm to (315.6, 156.7)
- moved S0:1 42.4 mm to (120.3, 75.7)
- moved S0:12 42.4 mm to (396.5, 75.7)
- moved S1:5 42.4 mm to (201.3, 99.5)
- moved S1:6 42.4 mm to (222.7, 99.5)
- moved S1:7 42.4 mm to (294.1, 99.5)
- moved S1:8 42.4 mm to (315.6, 99.5)
- moved C1 42.4 mm to (256.8, 232.9)
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Connections:
- IC2 pad 15: /CB3_1 -> /CB9_1
- IC3 pad 1: /CA3_2 -> /CA9_2
- IC3 pad 15: /CB3_2 -> /CB9_2
- IC4 pad 1: /CA3_3 -> /CA9_3
- IC4 pad 15: /CB3_3 -> /CB9_3
- S0:10 pad 7: /CB3_1 -> /CB9_1
- S0:11 pad 7: /CB3_1 -> /CB9_1
- S0:12 pad 7: /CB3_1 -> /CB9_1
- S0:7 pad 7: /CB3_1 -> /CB9_1
- S0:8 pad 7: /CB3_1 -> /CB9_1
- S0:9 pad 7: /CB3_1 -> /CB9_1
- S2:0 pad 7: /CA3_2 -> /CA9_2
- S2:1 pad 7: /CA3_2 -> /CA9_2
- S2:10 pad 7: /CB3_2 -> /CB9_2
- S2:11 pad 7: /CB3_2 -> /CB9_2
- S2:12 pad 7: /CB3_2 -> /CB9_2
- S2:13 pad 7: /CB3_2 -> /CB9_2
- S2:2 pad 7: /CA3_2 -> /CA9_2
- S2:3 pad 7: /CA3_2 -> /CA9_2
- S2:4 pad 7: /CA3_2 -> /CA9_2
- S2:5 pad 7: /CA3_2 -> /CA9_2
- S2:6 pad 7: /CA3_2 -> /CA9_2
- S2:7 pad 7: /CB3_2 -> /CB9_2
- S2:8 pad 7: /CB3_2 -> /CB9_2
- S2:9 pad 7: /CB3_2 -> /CB9_2
- S4:0 pad 7: /CA3_3 -> /CA9_3
- S4:1 pad 7: /CA3_3 -> /CA9_3
- S4:10 pad 7: /CB3_3 -> /CB9_3
- S4:11 pad 7: /CB3_3 -> /CB9_3
- S4:12 pad 7: /CB3_3 -> /CB9_3
- S4:13 pad 7: /CB3_3 -> /CB9_3
- S4:2 pad 7: /CA3_3 -> /CA9_3
- S4:3 pad 7: /CA3_3 -> /CA9_3
- S4:4 pad 7: /CA3_3 -> /CA9_3
- S4:5 pad 7: /CA3_3 -> /CA9_3
- S4:6 pad 7: /CA3_3 -> /CA9_3
- S4:7 pad 7: /CB3_3 -> /CB9_3
- S4:8 pad 7: /CB3_3 -> /CB9_3
- S4:9 pad 7: /CB3_3 -> /CB9_3
Routing:
- net /CB8_1: track 0.00 -> 276.7 mm, vias 0 -> 5
- net /R3: track 0.00 -> 252.8 mm
- net /R2: track 0.00 -> 252.8 mm
- net /R1: track 0.00 -> 252.8 mm
- net /R4: track 0.00 -> 252.8 mm
- net /CB7_1: track 0.00 -> 252.7 mm, vias 0 -> 3
- net /R5: track 0.00 -> 214.8 mm, vias 0 -> 2
- net /CB3_1: track 0.00 -> 205.1 mm, vias 0 -> 4
- net /CA7_2: track 0.00 -> 201.7 mm, vias 0 -> 2
- net /R0: track 0.00 -> 200.4 mm
- net /CA2_3: track 0.00 -> 192.9 mm, vias 0 -> 3
- net /CA3_3: track 0.00 -> 185.3 mm, vias 0 -> 3
- net /CA3_2: track 0.00 -> 183.8 mm, vias 0 -> 3
- net /CA7_1: track 0.00 -> 178.5 mm, vias 0 -> 2
- net /CB3_3: track 0.00 -> 177.9 mm, vias 0 -> 2
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
Commit message: lots of changes to pcb layout -- almost ready for rotation and final routing
Parts:
- added D0:7: D0:7, bwu-keyboard:SOD-123, F.Cu at (313.3, 74.4)
- added D1:7: D1:7, bwu-keyboard:SOD-123, F.Cu at (290.0, 100.7)
- added D2:7: D2:7, bwu-keyboard:SOD-123, F.Cu at (290.0, 108.7)
- added D3:7: D3:7, bwu-keyboard:SOD-123, F.Cu at (306.6, 138.8)
- added D4:7: D4:7, bwu-keyboard:SOD-123, F.Cu at (290.0, 155.0)
- S0:1, S0:10, S0:11, S0:12, S0:2, S0:3, S0:4, S0:5, S0:6, S0:8, S0:9, S1:1, S1:10, S1:11, S1:12, S1:2, S1:3, S1:4, S1:5, S1:6, S1:8, S1:9, S2:1, S2:10, S2:11, S2:12, S2:2, S2:3, S2:4, S2:5, S2:6, S2:8, S2:9, S3:1, S3:10, S3:11, S3:12, S3:2, S3:3, S3:4, S3:5, S3:6, S3:8, S3:9, S4:1, S4:10, S4:11, S4:12, S4:2, S4:3, S4:4, S4:5, S4:6, S4:8, S4:9, S5:1, S5:10, S5:11, S5:12, S5:2, S5:3, S5:4, S5:9: footprint bwu-keyboard:bwu-mx1a-1u-rgb -> bwu-keyboard:bwu-mx1a-1u-rgb-led-reverse
- S0:7, S1:7, S2:7, S3:7, S4:7: footprint bwu-keyboard:bwu-mx1a-1u-rgb -> bwu-keyboard:bwu-mx1a-1u-rgb-led-no-diode-reverse
- S1:0, S1:13, S2:0, S2:13, S3:0, S3:13, S4:0, S4:13, S5:0, S5:13: footprint bwu-keyboard:bwu-mx1a-150u-rgb -> bwu-keyboard:bwu-mx1a-150u-rgb-reverse
- S5:5, S5:6, S5:7, S5:8: footprint bwu-keyboard:bwu-mx1a-2u-rgb -> bwu-keyboard:bwu-mx1a-2u-rgb-reverse
- moved SW1 192.9 mm to (157.6, 83.1), turned to 180 degrees
- moved C8 184.6 mm to (256.5, 70.8), turned to 90 degrees
- moved C4 173.2 mm to (217.5, 84.9)
- moved C2 169.2 mm to (266.5, 70.3), turned to 90 degrees
- moved C7 167.1 mm to (302.4, 84.4)
- moved R2 163.8 mm to (259.4, 71.4), turned to 90 degrees
- moved C1 162.2 mm to (253.1, 70.8), turned to 90 degrees
- moved C6 156.5 mm to (302.3, 88.9)
- moved R1 156.3 mm to (262.9, 71.4), turned to 90 degrees
- moved C5 154.8 mm to (217.5, 87.1)
- moved Y1 149.4 mm to (212.0, 85.9)
- moved R3 148.0 mm to (265.7, 95.9)
- moved C3 145.4 mm to (256.8, 100.2), turned to 270 degrees
- moved IC1 133.6 mm to (260.0, 85.0), turned to 270 degrees
- moved R4 125.4 mm to (267.0, 127.0), turned to 270 degrees
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Connections:
- CON1 pad 4: (no net) -> Net-(CON1-Pad4)
- IC1 pad 1: /R1 -> /R0
- IC1 pad 10: /C9 -> /R3
- IC1 pad 11: /CA -> /R4
- IC1 pad 12: (no net) -> /R5
- IC1 pad 20: /CB -> Net-(IC1-Pad20)
- IC1 pad 21: /CC -> Net-(IC1-Pad21)
- IC1 pad 22: /CD -> /C0
- IC1 pad 25: /R5 -> /C1
- IC1 pad 26: /C6 -> /C2
- IC1 pad 27: /C7 -> /C3
- IC1 pad 28: /C0 -> /C4
- IC1 pad 29: (no net) -> /C5
- IC1 pad 30: (no net) -> /C6
- IC1 pad 31: /C1 -> /SDB
- IC1 pad 32: /C2 -> /C7
- IC1 pad 36: /C3 -> /C8
- IC1 pad 37: /C4 -> /C9
- IC1 pad 38: /C5 -> /CA
- IC1 pad 39: /R4 -> /CB
- IC1 pad 40: /R3 -> /CC
- IC1 pad 41: /R2 -> /CD
- IC1 pad 8: /C8 -> /R1
- IC1 pad 9: /R0 -> /R2
- IC2 pad 16: (no net) -> Net-(IC2-Pad16)
- IC2 pad 17: (no net) -> Net-(IC2-Pad17)
- IC2 pad 4: (no net) -> Net-(IC2-Pad4)
- IC3 pad 16: (no net) -> Net-(IC3-Pad16)
- IC3 pad 17: (no net) -> Net-(IC3-Pad17)
- IC3 pad 4: (no net) -> Net-(IC3-Pad4)
- IC4 pad 16: (no net) -> Net-(IC4-Pad16)
- IC4 pad 17: (no net) -> Net-(IC4-Pad17)
- IC4 pad 4: (no net) -> Net-(IC4-Pad4)
- SW1 pad 1: (no net) -> Net-(SW1-Pad1)
Routing:
- net /R5: track 214.8 -> 622.3 mm, vias 2 -> 4
- net /R4: track 252.8 -> 649.3 mm, vias 0 -> 4
- net /R3: track 252.8 -> 616.1 mm, vias 0 -> 4
- net /R2: track 252.8 -> 582.9 mm, vias 0 -> 5
- net /R1: track 252.8 -> 546.8 mm, vias 0 -> 3
- net /R0: track 200.4 -> 486.6 mm, vias 0 -> 2
- net /C0: track 82.9 -> 223.5 mm
- net /CD: track 88.8 -> 213.2 mm, vias 5 -> 6
- net /C1: track 135.6 -> 248.8 mm, vias 6 -> 7
- net /CA2_3: track 192.9 -> 303.2 mm, vias 3 -> 1
- net /CA3_3: track 185.3 -> 280.3 mm, vias 3 -> 2
- net /CA1_3: track 171.5 -> 264.2 mm, vias 3 -> 2
- net /C2: track 127.3 -> 217.7 mm, vias 6 -> 7
- net /CC: track 117.2 -> 206.4 mm, vias 6 -> 7
- net /CB7_2: track 173.0 -> 253.7 mm, vias 3 -> 1
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