File: gaia/gaia2.kicad_pcb (KiCad board)
At the start: 2 copper layers, 360 x 170 mm, 108 parts, among them CON1 USB-MINI-B WM17115-ND, IC1 ATMEGA32U4, IC2 IS31FL3731, IC3 IS31FL3731, IC4 IS31FL3731, SW1 SW423CT-ND, Y1 16MHz

Commit message: checkpointing
Parts:
- moved S5:6 17.8 mm to (226.0, 197.0), turned to 60 degrees
- moved S5:7 17.8 mm to (294.8, 197.0), turned to 300 degrees
- moved S5:5 11.0 mm to (209.5, 187.5), turned to 60 degrees
- moved S5:8 11.0 mm to (311.3, 187.5), turned to 300 degrees
Routing:
- net /R5: track 659.7 -> 717.0 mm
- net /CB2_3: track 195.9 -> 228.8 mm
- net /C7: track 148.7 -> 180.7 mm
- net /C5: track 139.0 -> 168.4 mm
- net /CB3_3: track 221.5 -> 247.2 mm
- net /CA7_3: track 167.7 -> 188.2 mm
- net /CB4_3: track 147.2 -> 166.4 mm
- net /C6: track 142.9 -> 159.7 mm
- net /C8: track 89.7 -> 104.9 mm
- net /CA8_3: track 194.4 -> 208.8 mm
- net /CA3_3: track 250.9 -> 263.1 mm
- net /CA1_3: track 220.9 -> 229.7 mm
- net /CB1_3: track 218.8 -> 225.3 mm
- net /CA2_3: track 275.7 -> 282.3 mm
